Commit message: smartcar can move in gazebo

File: urdf/smart_car.urdf (robot description, URDF)
Before this commit: robot smartcar, 7 links, 6 joints
Links:
- removed link stl_link
- added link base_footprint; visual box size=0.001 0.001 0.001
- link base_link: mass None -> 10; geometry collision box size=0.25 .16 .05; visual box size=0.25 .16 .05
- link head: mass None -> 1; geometry collision box size=.02 .03 .03; visual box size=.02 .03 .03
- link left_back_wheel: mass None -> 1; geometry collision cylinder length=.02 radius=0.025; visual cylinder length=.02 radius=0.025
- link left_front_wheel: mass None -> 1; geometry collision cylinder length=.02 radius=0.025; visual cylinder length=.02 radius=0.025
- link right_back_wheel: mass None -> 1; geometry collision cylinder length=.02 radius=0.025; visual cylinder length=.02 radius=0.025
- link right_front_wheel: mass None -> 1; geometry collision cylinder length=.02 radius=0.025; visual cylinder length=.02 radius=0.025
Joints:
- removed joint stl_joint
- added joint base_footprint_joint: type fixed, parent base_footprint, child base_link, origin xyz=0 0 0.05 rpy=0 0 0
- joint left_back_wheel_joint: origin xyz=-0.08 -0.1 0.025 rpy=0 1.57075 0 -> xyz=-0.08 0.085 -0.025 rpy=1.57 0 0
- joint left_front_wheel_joint: origin xyz=-0.08 0.1 0.025 rpy=0 1.57075 0 -> xyz=0.08 0.085 -0.025 rpy=1.57 0 0
- joint right_back_wheel_joint: origin xyz=0.08 -0.1 0.025 rpy=0 1.57075 0 -> xyz=-0.08 -0.085 -0.025 rpy=1.57 0 0
- joint right_front_wheel_joint: origin xyz=0.08 0.1 0.025 rpy=0 1.57075 0 -> xyz=0.08 -0.085 -0.025 rpy=1.57 0 0
- joint tobox: origin xyz=0 0.08 0.09 -> xyz=0.1 0 0.04

Commit message: 修复运动反向的问题

File: urdf/smart_car.urdf (robot description, URDF)
Before this commit: robot smartcar, 7 links, 6 joints
Joints:
- joint left_back_wheel_joint: origin xyz=-0.08 0.085 -0.025 rpy=1.57 0 0 -> xyz=-0.08 0.085 -0.025 rpy=-1.57 0 0
- joint left_front_wheel_joint: origin xyz=0.08 0.085 -0.025 rpy=1.57 0 0 -> xyz=0.08 0.085 -0.025 rpy=-1.57 0 0
- joint right_back_wheel_joint: origin xyz=-0.08 -0.085 -0.025 rpy=1.57 0 0 -> xyz=-0.08 -0.085 -0.025 rpy=-1.57 0 0
- joint right_front_wheel_joint: origin xyz=0.08 -0.085 -0.025 rpy=1.57 0 0 -> xyz=0.08 -0.085 -0.025 rpy=-1.57 0 0
